Commit message: added xacro with variables and proper math

File: src/robot_description/urdf/lebot.urdf (robot description, URDF)
Before this commit: robot service_bot, 10 links, 9 joints
Joints:
- joint base_left_support_wheel_joint: axis (none) -> 0 0 1; type fixed -> continuous
- joint base_right_support_wheel_joint: axis (none) -> 0 0 1; type fixed -> continuous
