Commit message: added collisions

File: src/robot_description/urdf/lebot.urdf.xacro (robot description, xacro)
@@ -42,6 +42,6 @@
             </material>
         </visual>
-        <!-- <collision/>
-        <inertial />-->
+        <collision><geometry><box size="${base_depth} ${base_width} ${base_height}"/></geometry></collision>
+        <!--inertial />-->
     </link>
     <link name="left_wheel_link">
@@ -53,6 +53,6 @@
             <material name="red"/>
         </visual>
-       <!-- <collision/>
-        <inertial />-->
+       <collision><geometry><cylinder radius="${drive_wheel_rad}" length="${wheel_len}"/></geometry></collision>
+        <!--inertial />-->
     </link>
     <link name="right_wheel_link">
@@ -64,6 +64,6 @@
             <material name="red"/>
         </visual>
-        <!--<collision/>
-        <inertial />-->
+        <collision><geometry><cylinder radius="${drive_wheel_rad}" length="${wheel_len}"/></geometry></collision>
+        <!--inertial />-->
     </link>
     <link name="right_support_wheel_link">
@@ -75,6 +75,6 @@
             <material name="green"/>
         </visual>
-        <!--<collision/>
-        <inertial />-->
+        <collision><geometry><cylinder radius="${supp_wheel_rad}" length="${wheel_len}"/></geometry></collision>
+        <!--inertial />-->
     </link>
     <link name="left_support_wheel_link">
@@ -86,6 +86,6 @@
             <material name="green"/>
         </visual>
-        <!--<collision/>
-        <inertial />-->
+        <collision><geometry><cylinder radius="${supp_wheel_rad}" length="${wheel_len}"/></geometry></collision>
+        <!--inertial />-->
     </link>
     <link name="left_support_link">
@@ -97,6 +97,6 @@
             <material name="teal"/>
         </visual>
-        <!--collision/>3
-        <inertial /-->
+        <collision><geometry><box size="${side_block_depth} ${side_block_width} ${side_block_height}"/></geometry></collision>
+        <!--inertial /-->
     </link>
     <link name="right_support_link">
@@ -108,6 +108,6 @@
             <material name="teal"/>
         </visual>
-        <!--collision/>
-        <inertial /-->
+        <collision><geometry><box size="${side_block_depth} ${side_block_width} ${side_block_height}"/></geometry></collision>
+        <!--inertial /-->
     </link>
     <link name="top_block_link">
@@ -119,6 +119,6 @@
             <material name="teal"/>
         </visual>
-        <!--collision/>
-        <inertial /-->
+        <collision><geometry><box size="${top_block_depth} ${top_block_width} ${top_block_height}"/></geometry></collision>/>
+        <!--inertial /-->
     </link>
     <link name="lidar_link">
@@ -130,6 +130,6 @@
             <material name="white"/>
         </visual>
-        <!--collision/>
-        <inertial /-->
+        <collision><geometry><cylinder radius="${sensor_rad}" length="${sensor_len}"/></geometry></collision>
+        <!--inertial /-->
     </link>
     <link name="camera_link">
@@ -141,6 +141,6 @@
             <material name="white"/>
         </visual>
-        <!--collision/>
-        <inertial /-->
+        <collision><geometry><cylinder radius="${sensor_rad}" length="${sensor_len}"/></geometry></collision>/>
+        <!--inertial /-->
     </link>
     <joint name="base_left_wheel_joint" type="continuous">

Commit message: added inerti

File: src/robot_description/urdf/lebot.urdf.xacro (robot description, xacro)
@@ -4,19 +4,25 @@
     <xacro:property name="base_height" value=".125"/>
     <xacro:property name="base_depth" value=".45"/>
+    <xacro:property name="base_mass" value="2.0"/>
     <xacro:property name="top_block_width" value=".50"/>
     <xacro:property name="top_block_height" value="0.20"/>
     <xacro:property name="top_block_depth" value="0.10"/>
+    <xacro:property name="top_block_mass" value="0.5"/>
     <xacro:property name="side_block_width" value="0.050"/>
     <xacro:property name="side_block_height" value="${1.10-(top_block_height-base_height)}"/>
     <xacro:property name="side_block_depth" value="0.10"/>
+    <xacro:property name="support_mass" value="0.3"/>
     <xacro:property name="drive_wheel_rad" value=".055"/>
+    <xacro:property name="wheel_mass" value="0.2"/>
     <xacro:property name="wheel_len" value=".01"/>
     <xacro:property name="supp_wheel_rad" value=".03"/>
+    <xacro:property name="supp_wheel_mass" value="0.1"/>
     <xacro:property name="wheel_offset" value=".01"/>
     <xacro:property name="drive_wheel_posZ" value="-${(((base_height/2)+wheel_offset)-(drive_wheel_rad*2))+(drive_wheel_rad)}"/>
-    <xacro:property name="supp_whell_posZ" value="-${(((base_height/2)+wheel_offset)-(supp_wheel_rad*2))+(supp_wheel_rad)}"/>
-    <xacro:property name="whell_posY" value="${base_width/2 + wheel_len/2}"/>
+    <xacro:property name="supp_wheel_posZ" value="-${(((base_height/2)+wheel_offset)-(supp_wheel_rad*2))+(supp_wheel_rad)}"/>
+    <xacro:property name="wheel_posY" value="${base_width/2 + wheel_len/2}"/>
     <xacro:property name="sensor_rad" value=".03"/>
     <xacro:property name="sensor_len" value=".03"/>
+    <xacro:property name="sensor_mass" value="0.05"/>
     <xacro:property name="PI" value="3.1415"/>
     <material name="red">
@@ -43,5 +49,13 @@
         </visual>
         <collision><geometry><box size="${base_depth} ${base_width} ${base_height}"/></geometry></collision>
-        <!--inertial />-->
+        <inertial>
+            <origin xyz="0 0 0" rpy="0 0 0"/>
+            <mass value="${base_mass}"/>
+            <inertia
+                ixx="${base_mass/12.0 * (base_width*base_width + base_height*base_height)}"
+                iyy="${base_mass/12.0 * (base_depth*base_depth + base_height*base_height)}"
+                izz="${base_mass/12.0 * (base_depth*base_depth + base_width*base_width)}"
+                ixy="0" ixz="0" iyz="0"/>
+        </inertial>
     </link>
     <link name="left_wheel_link">
@@ -54,5 +68,13 @@
         </visual>
        <collision><geometry><cylinder radius="${drive_wheel_rad}" length="${wheel_len}"/></geometry></collision>
-        <!--inertial />-->
+       <inertial>
+            <origin xyz="0 0 0" rpy="0 0 0"/>
+            <mass value="${wheel_mass}"/>
+            <inertia
+                ixx="${wheel_mass/12.0 * (3*drive_wheel_rad*drive_wheel_rad + wheel_len*wheel_len)}"
+                iyy="${wheel_mass/12.0 * (3*drive_wheel_rad*drive_wheel_rad + wheel_len*wheel_len)}"
+                izz="${wheel_mass/2.0 * drive_wheel_rad*drive_wheel_rad}"
+                ixy="0" ixz="0" iyz="0"/>
+        </inertial>
     </link>
     <link name="right_wheel_link">
@@ -65,5 +87,13 @@
         </visual>
         <collision><geometry><cylinder radius="${drive_wheel_rad}" length="${wheel_len}"/></geometry></collision>
-        <!--inertial />-->
+        <inertial>
+            <origin xyz="0 0 0" rpy="0 0 0"/>
+            <mass value="${wheel_mass}"/>
+            <inertia
+                ixx="${wheel_mass/12.0 * (3*drive_wheel_rad*drive_wheel_rad + wheel_len*wheel_len)}"
+                iyy="${wheel_mass/12.0 * (3*drive_wheel_rad*drive_wheel_rad + wheel_len*wheel_len)}"
+                izz="${wheel_mass/2.0 * drive_wheel_rad*drive_wheel_rad}"
+                ixy="0" ixz="0" iyz="0"/>
+        </inertial>
     </link>
     <link name="right_support_wheel_link">
@@ -76,5 +106,13 @@
         </visual>
         <collision><geometry><cylinder radius="${supp_wheel_rad}" length="${wheel_len}"/></geometry></collision>
-        <!--inertial />-->
+        <inertial>
+            <origin xyz="0 0 0" rpy="0 0 0"/>
+            <mass value="${supp_wheel_mass}"/>
+            <inertia
+                ixx="${supp_wheel_mass/12.0 * (3*supp_wheel_rad*supp_wheel_rad + wheel_len*wheel_len)}"
+                iyy="${supp_wheel_mass/12.0 * (3*supp_wheel_rad*supp_wheel_rad + wheel_len*wheel_len)}"
+                izz="${supp_wheel_mass/2.0 * supp_wheel_rad*supp_wheel_rad}"
+                ixy="0" ixz="0" iyz="0"/>
+        </inertial>
     </link>
     <link name="left_support_wheel_link">
@@ -87,5 +125,13 @@
         </visual>
         <collision><geometry><cylinder radius="${supp_wheel_rad}" length="${wheel_len}"/></geometry></collision>
-        <!--inertial />-->
+        <inertial>
+            <origin xyz="0 0 0" rpy="0 0 0"/>
+            <mass value="${supp_wheel_mass}"/>
+            <inertia
+                ixx="${supp_wheel_mass/12.0 * (3*supp_wheel_rad*supp_wheel_rad + wheel_len*wheel_len)}"
+                iyy="${supp_wheel_mass/12.0 * (3*supp_wheel_rad*supp_wheel_rad + wheel_len*wheel_len)}"
+                izz="${supp_wheel_mass/2.0 * supp_wheel_rad*supp_wheel_rad}"
+                ixy="0" ixz="0" iyz="0"/>
+        </inertial>
     </link>
     <link name="left_support_link">
@@ -98,5 +144,13 @@
         </visual>
         <collision><geometry><box size="${side_block_depth} ${side_block_width} ${side_block_height}"/></geometry></collision>
-        <!--inertial /-->
+        <inertial>
+            <origin xyz="0 0 0" rpy="0 0 0"/>
+            <mass value="${support_mass}"/>
+            <inertia
+                ixx="${support_mass/12.0 * (side_block_width*side_block_width + side_block_height*side_block_height)}"
+                iyy="${support_mass/12.0 * (side_block_depth*side_block_depth + side_block_height*side_block_height)}"
+                izz="${support_mass/12.0 * (side_block_depth*side_block_depth + side_block_width*side_block_width)}"
+                ixy="0" ixz="0" iyz="0"/>
+        </inertial>
     </link>
     <link name="right_support_link">
@@ -109,5 +163,13 @@
         </visual>
         <collision><geometry><box size="${side_block_depth} ${side_block_width} ${side_block_height}"/></geometry></collision>
-        <!--inertial /-->
+        <inertial>
+            <origin xyz="0 0 0" rpy="0 0 0"/>
+            <mass value="${support_mass}"/>
+            <inertia
+                ixx="${support_mass/12.0 * (side_block_width*side_block_width + side_block_height*side_block_height)}"
+                iyy="${support_mass/12.0 * (side_block_depth*side_block_depth + side_block_height*side_block_height)}"
+                izz="${support_mass/12.0 * (side_block_depth*side_block_depth + side_block_width*side_block_width)}"
+                ixy="0" ixz="0" iyz="0"/>
+        </inertial>
     </link>
     <link name="top_block_link">
@@ -120,5 +182,13 @@
         </visual>
         <collision><geometry><box size="${top_block_depth} ${top_block_width} ${top_block_height}"/></geometry></collision>/>
-        <!--inertial /-->
+        <inertial>
+            <origin xyz="0 0 0" rpy="0 0 0"/>
+            <mass value="${top_block_mass}"/>
+            <inertia
+                ixx="${top_block_mass/12.0 * (top_block_width*top_block_width + top_block_height*top_block_height)}"
+                iyy="${top_block_mass/12.0 * (top_block_depth*top_block_depth + top_block_height*top_block_height)}"
+                izz="${top_block_mass/12.0 * (top_block_depth*top_block_depth + top_block_width*top_block_width)}"
+                ixy="0" ixz="0" iyz="0"/>
+        </inertial>
     </link>
     <link name="lidar_link">
@@ -131,5 +201,13 @@
         </visual>
         <collision><geometry><cylinder radius="${sensor_rad}" length="${sensor_len}"/></geometry></collision>
-        <!--inertial /-->
+        <inertial>
+            <origin xyz="0 0 0" rpy="0 0 0"/>
+            <mass value="${sensor_mass}"/>
+            <inertia
+                ixx="${sensor_mass/12.0 * (3*sensor_rad*sensor_rad + sensor_len*sensor_len)}"
+                iyy="${sensor_mass/12.0 * (3*sensor_rad*sensor_rad + sensor_len*sensor_len)}"
+                izz="${sensor_mass/2.0 * sensor_rad*sensor_rad}"
+                ixy="0" ixz="0" iyz="0"/>
+        </inertial>
     </link>
     <link name="camera_link">
@@ -142,10 +220,18 @@
         </visual>
         <collision><geometry><cylinder radius="${sensor_rad}" length="${sensor_len}"/></geometry></collision>/>
-        <!--inertial /-->
+        <inertial>
+            <origin xyz="0 0 0" rpy="0 0 0"/>
+            <mass value="${sensor_mass}"/>
+            <inertia
+                ixx="${sensor_mass/12.0 * (3*sensor_rad*sensor_rad + sensor_len*sensor_len)}"
+                iyy="${sensor_mass/12.0 * (3*sensor_rad*sensor_rad + sensor_len*sensor_len)}"
+                izz="${sensor_mass/2.0 * sensor_rad*sensor_rad}"
+                ixy="0" ixz="0" iyz="0"/>
+        </inertial>
     </link>
     <joint name="base_left_wheel_joint" type="continuous">
         <parent link="base_link"/>
         <child link="left_wheel_link"/>
-        <origin xyz="-0.13 ${whell_posY} ${drive_wheel_posZ}" rpy="${PI/2.0} 0 0"/>
+        <origin xyz="-0.13 ${wheel_posY} ${drive_wheel_posZ}" rpy="${PI/2.0} 0 0"/>
         <axis xyz="0 0 1" />
     </joint>
@@ -153,5 +239,5 @@
         <parent link="base_link"/>
         <child link="left_support_wheel_link"/>
-        <origin xyz="0.13 ${whell_posY} ${supp_whell_posZ}" rpy="${PI/2.0} 0 0"/>
+        <origin xyz="0.13 ${wheel_posY} ${supp_wheel_posZ}" rpy="${PI/2.0} 0 0"/>
         <axis xyz="0 0 1" />
     </joint>
@@ -159,5 +245,5 @@
         <parent link="base_link"/>
         <child link="right_wheel_link"/>
-        <origin xyz="-0.13 -${whell_posY} ${drive_wheel_posZ}" rpy="${PI/2.0} 0 0"/>
+        <origin xyz="-0.13 -${wheel_posY} ${drive_wheel_posZ}" rpy="${PI/2.0} 0 0"/>
         <axis xyz="0 0 1" />
     </joint>
@@ -165,5 +251,5 @@
         <parent link="base_link"/>
         <child link="right_support_wheel_link"/>
-        <origin xyz="0.13 -${whell_posY} ${supp_whell_posZ}" rpy="${PI/2.0} 0 0"/>
+        <origin xyz="0.13 -${wheel_posY} ${supp_wheel_posZ}" rpy="${PI/2.0} 0 0"/>
         <axis xyz="0 0 1" />
     </joint>
@@ -198,4 +284,3 @@
         <!--axis xyz="0 0 1" /-->
     </joint>
-<!-- 2 - 1.1875 -->
 </robot>
